File: electronics/apico_shield/apico_shield.kicad_pcb (KiCad board)
At the start: 2 copper layers, 68.6 x 53.3 mm, 6 parts

Commit message: updated pcb
Parts:
- added J1: Power out, Connector_PinHeader_2.54mm:PinHeader_1x02_P2.54mm_Vertical, F.Cu at (119.4, 78.7)
- C1: value Grove CO2,T,RH -> Grove CO2
- b1: value LORA Radio -> Radio rfm9x
Connections:
- C2 pad 1: Net-(APICO_UNO1-Pad5V1) -> Net-(C2-Pad1)
- C3 pad 2: Net-(APICO_UNO1-Pad5V1) -> Net-(C2-Pad1)
Routing:
- net Net-(C2-Pad1): track 0.00 -> 43.1 mm
- net Net-(APICO_UNO1-Pad5V1): track 126.3 -> 95.1 mm
- net Net-(APICO_UNO1-PadGND1): track 115.7 -> 126.5 mm
- net Net-(APICO_UNO1-PadD9): track 40.8 -> 47.1 mm
- net Net-(APICO_UNO1-PadD8): track 49.5 -> 43.5 mm
- net Net-(APICO_UNO1-PadD12): track 43.8 -> 49.4 mm
- net Net-(APICO_UNO1-PadD11): track 49.5 -> 53.4 mm
- net Net-(APICO_UNO1-PadD7): track 54.3 -> 56.3 mm
Other:
- board text added: "ApiCo Shield v1.1"
- board text removed: "ApiCo Shield v1.0"
