File: electronics/apico_shield/apico_shield.sch (KiCad schematic (older format))
At the start: 6 parts

Commit message: updated pcb
Parts:
- added J1: Power out, Connector_PinHeader_2.54mm:PinHeader_1x02_P2.54mm_Vertical, symbol Connector:Conn_01x02_Male
Connections:
- net at APICO_UNO1.5V1 (5V), C1.2 (Pin_2), b1.9 (Pin_9)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: now also J1.2 (Pin_2); no longer C2.1 (Pin_1), C3.2 (Pin_2)
- new net: C2.1 (Pin_1), C3.2 (Pin_2), J1.1 (Pin_1)
Changed lines of the file:
@@
 	7900 3700 7900 5150
 Wire Wire Line
-	7900 5150 3850 5150
+	7900 5150 3900 5150
 Connection ~ 7900 3700
 Wire Wire Line
@@
 Wire Wire Line
 	3400 3150 3850 3150
-Wire Wire Line
-	3850 3150 3850 4200
-Connection ~ 3850 4600
 $Comp
 L Connector:Conn_01x05_Male C2
@@
 $EndComp
 Wire Wire Line
-	3450 4200 3850 4200
-Connection ~ 3850 4200
-Wire Wire Line
-	3850 4200 3850 4600
+	3450 4200 3700 4200
 Wire Wire Line
 	3450 4300 3950 4300
@@
 	4150 3300 4450 3300
 Wire Wire Line
-	3850 4600 3850 5150
-Wire Wire Line
 	3450 5050 3950 5050
 Connection ~ 3950 5050
@@
 	3450 5150 3700 5150
 Wire Wire Line
-	3700 5150 3700 4600
+	3700 4200 3700 5150
 Wire Wire Line
-	3700 4600 3850 4600
+	3850 3150 3850 4600
+Wire Wire Line
+	3850 4600 3850 5150
+Connection ~ 3850 4600
+$Comp
+L Connector:Conn_01x02_Male J1
+U 1 1 6187056D
+P 3800 5750
+F 0 "J1" V 3954 5562 50  0000 R CNN
+F 1 "Power out" V 3863 5562 50  0000 R CNN
+F 2 "Connector_PinHeader_2.54mm:PinHeader_1x02_P2.54mm_Vertical" H 3800 5750 50  0001 C CNN
+F 3 "~" H 3800 5750 50  0001 C CNN
+	1    3800 5750
+	0    -1   -1   0
+$EndComp
+Wire Wire Line
+	3800 5550 3800 5300
+Wire Wire Line
+	3800 5300 3700 5300
+Wire Wire Line
+	3700 5300 3700 5150
+Connection ~ 3700 5150
+Wire Wire Line
+	3900 5550 3900 5150
+Connection ~ 3900 5150
+Wire Wire Line
+	3900 5150 3850 5150
 $EndSCHEMATC
